Commit message: maybe working with new urdf ???

File: awd/data/assets/mini2_bdx/mini2_bdx.urdf (robot description, URDF)
Before this commit: robot onshape, 18 links, 17 joints
Links:
- removed link head_pitch_assembly
- removed link neck_assembly
- added link head_pitch_to_yaw, mass 0.016937787992336000853; collision mesh filename=./head_pitch_to_yaw.stl; visual mesh filename=./head_pitch_to_yaw.stl
- added link left_antenna_holder, mass 0.00421628909577088061; collision mesh filename=./antenna.stl; collision mesh filename=./left_antenna_holder.stl
- added link neck_pitch_assembly, mass 0.066180000000000016591; collision mesh filename=./drive_palonier.stl; collision mesh filename=./neck_left_sheet.stl
- added link neck_yaw_assembly, mass 0.091809888579250376051; collision mesh filename=./drive_palonier.stl; collision mesh filename=./head_yaw_to_roll.stl
- added link right_antenna_holder, mass 0.0042162869849506796893; collision mesh filename=./antenna.stl; collision mesh filename=./right_antenna_holder.stl
- link foot_assembly: mass 0.056240000000000012204 -> 0.075240000000000015201; geometry collision mesh filename=./foot_bottom_pla.stl; collision mesh filename=./foot_bottom_tpu.stl
- link foot_assembly_2: mass 0.056240000000000012204 -> 0.075240000000000015201; geometry collision mesh filename=./foot_bottom_pla.stl; collision mesh filename=./foot_bottom_tpu.stl
- link head_assembly: mass 0.22929000000000004933 -> 0.35258298534369525434; geometry collision mesh filename=./board.stl; collision mesh filename=./drive_palonier.stl
- link hip_roll_assembly: geometry collision mesh filename=./drive_palonier.stl; collision mesh filename=./passive_palonier.stl
- link hip_roll_assembly_2: geometry collision mesh filename=./drive_palonier.stl; collision mesh filename=./passive_palonier.stl
- link knee_and_ankle_assembly: mass 0.12406999999999994422 -> 0.12407000000000001361; geometry collision mesh filename=./drive_palonier.stl; collision mesh filename=./left_cache.stl
- link knee_and_ankle_assembly_2: geometry collision mesh filename=./drive_palonier.stl; collision mesh filename=./left_knee_to_ankle_left_sheet.stl
- link knee_and_ankle_assembly_3: mass 0.12407000000000002748 -> 0.12407000000000004136; geometry collision mesh filename=./drive_palonier.stl; collision mesh filename=./left_knee_to_ankle_left_sheet.stl
- link knee_and_ankle_assembly_4: geometry collision mesh filename=./drive_palonier.stl; collision mesh filename=./left_knee_to_ankle_left_sheet.stl
- link left_roll_to_pitch_assembly: mass 0.075160000000000018461 -> 0.075160000000000004583; geometry collision mesh filename=./drive_palonier.stl; collision mesh filename=./left_roll_to_pitch.stl
- link right_roll_to_pitch_assembly: mass 0.075160000000000018461 -> 0.075160000000000004583; geometry collision mesh filename=./drive_palonier.stl; collision mesh filename=./passive_palonier.stl
- link trunk_assembly: mass 0.55922072109020470876 -> 0.69852641931996084512; geometry collision mesh filename=./battery_pack_lid.stl; collision mesh filename=./bms.stl
Joints:
- added joint head_roll: type revolute, parent neck_yaw_assembly, child head_assembly, origin xyz=0.040950000000000000289 -4.2214766838438722019e-16 -0.019149999999999833822 rpy=1.2411687278497551329e-14 -1.5707963267948830133 0, axis 0 0 1, limit lower=-0.52359877559829881566 upper=0.52359877559829881566 effort=1 velocity=20
- added joint left_antenna: type revolute, parent head_assembly, child left_antenna_holder, origin xyz=0.00070406945503187490232 0.060662837687359048855 0.1164348532954449511 rpy=-3.1415926535897802374 1.3045791727887245948 1.3234423712230847237, axis 0 0 1, limit lower=-1.570796326794896558 upper=1.570796326794896558 effort=1 velocity=20
- added joint right_antenna: type revolute, parent head_assembly, child right_antenna_holder, origin xyz=0.00070406945503675988363 -0.060662837687358986405 0.11643485329544003837 rpy=-3.1415926535897802374 1.3045791727887252609 -1.3234423712230598547, axis 0 0 1, limit lower=-1.570796326794896558 upper=1.570796326794896558 effort=1 velocity=20
- joint head_frame: origin xyz=4.1633363423443370266e-17 0 -0.01249999999999990008 rpy=-3.1415926535897797933 4.3716373664754018489e-18 7.4988647406086779923e-30 -> xyz=0.04244999999999957141 2.135878279796443735e-17 0.035950000000000377487 rpy=-0 1.570796326794896558 0
- joint head_pitch: child head_pitch_assembly -> head_pitch_to_yaw; limit lower=-1.570796326794896558 upper=1.570796326794896558 effort=1 velocity=20 -> lower=-0.785398163397448279 upper=0.785398163397448279 effort=1 velocity=20; origin xyz=1.0408340855860842566e-16 0.066000000000000391687 -3.4694469519536141888e-18 rpy=-1.0915849447069766081e-16 -7.3845547632106068786e-17 -1.0417200973690603325e-16 -> xyz=-5.42101086242752217e-17 0.066000000000000086375 -1.0408340855860842566e-17 rpy=-1.9479487599482720301e-16 -1.1423136863502905442e-16 1.7347234747146296461e-18; parent neck_assembly -> neck_pitch_assembly
- joint head_yaw: child head_assembly -> neck_yaw_assembly; limit lower=-2.9670597283903603625 upper=2.9670597283903603625 effort=1 velocity=20 -> lower=-2.7925268031909271649 upper=2.7925268031909271649 effort=1 velocity=20; origin xyz=-2.0816681711721685133e-17 0.056900000000000033884 0.019049999999999952388 rpy=1.5707963267948958919 -2.9140480977164958126e-15 -8.9523033089878119206e-15 -> xyz=-9.9746599868666407929e-18 0.056999999999999967359 0.019050000000000014838 rpy=-1.570796326794896558 -1.3706437208012195828e-25 6.1232339958582419871e-17; parent head_pitch_assembly -> head_pitch_to_yaw
- joint left_ankle: origin xyz=0 -0.07865000000000006708 9.9999999999988986588e-05 rpy=-5.5077724532749743024e-16 9.2653469445928301633e-16 3.2402024558001311503e-14 -> xyz=-7.9103390504542403505e-16 -0.078649999999999428701 9.9999999999794697558e-05 rpy=1.636340693842024721e-16 1.1379785959205303308e-15 -2.7755597583208935156e-17
- joint left_foot_frame: origin xyz=0 -0.036724999999999979883 0.019049999999999983613 rpy=-1.570796326794896558 -3.4146152368508307717e-19 -1.8519077370852487142e-17 -> xyz=0.00049999999999995187183 -0.036224999999999729638 0.019550000000000331002 rpy=-1.570796326794896558 4.8789097652664912905e-18 2.353432088828639061e-23
- joint left_hip_pitch: limit lower=-1.570796326794896558 upper=0.52359877559829881566 effort=1 velocity=20 -> lower=-1.2217304763960306069 upper=0.52359877559829881566 effort=1 velocity=20; origin xyz=0.074149999999998272848 1.249000902703301108e-15 0.035109999999998510456 rpy=3.1415926535897926719 1.5707963267948574781 0 -> xyz=0.074149999999999799405 -1.9529191631895148618e-17 0.035109999999999898235 rpy=3.141592653589793116 1.570796326794896336 0
- joint left_hip_roll: origin xyz=0.019050000000002648148 1.9602375278537920167e-15 -0.046015000000004538383 rpy=-1.5707963267950215691 1.6937530152664249305e-13 1.5707963267952902431 -> xyz=0.019050000000003588368 4.3576253716537394212e-15 -0.046015000000001519964 rpy=-1.5707963267949396347 9.7936145200150713608e-14 1.5707963267946445374
- joint left_hip_yaw: origin xyz=-0.056394334796673495358 0.028602766445326346934 0.024395090932709764808 rpy=-6.2403804745132919901e-14 0.021825623709755430368 1.3218914061185209833e-13 -> xyz=-0.018999999999998434808 0.035000000000000974776 0.04594093881237738819 rpy=-1.5205902553582758499e-16 -2.2037927038784495587e-14 -6.3658912806794774433e-27
- joint left_knee: origin xyz=-9.7144514654701197287e-17 -0.078649999999999734013 9.9999999999961231012e-05 rpy=7.358361518165846965e-16 5.0845139115396107043e-16 -7.1846367703695162136e-14 -> xyz=-2.9837243786801082024e-16 -0.078650000000000871991 9.99999999999751088e-05 rpy=-2.6413758326899544516e-16 -7.0075679691128679348e-24 -2.4877517507049828295e-26
- joint neck_pitch: child neck_assembly -> neck_pitch_assembly; origin xyz=-0.035437537550831413324 0.012752766445331959258 0.068008119366846808695 rpy=1.5707963267948341635 0.021825623709755184038 1.3218913913091132832e-13 -> xyz=0.00099999999999899474856 0.019150000000000326483 0.090000938812376224396 rpy=1.57079632679489678 -2.2204460492503130808e-14 6.1232449680326617825e-17
- joint right_ankle: origin xyz=-2.7755575615628913511e-17 -0.078650000000000080957 9.9999999999961231012e-05 rpy=-2.6194324489465746712e-16 2.8316471284964215798e-29 9.5878895885319479181e-14 -> xyz=1.3877787807814456755e-17 -0.078649999999999928302 0.00010000000000004449774 rpy=-2.6413812280837946538e-16 -1.7764738567684265366e-22 4.6805027693161558698e-25
- joint right_foot_frame: origin xyz=-1.3877787807814456755e-17 -0.036724999999999979883 0.019049999999999969735 rpy=-1.570796326794896558 -4.7247190275601867229e-17 6.0085748048618062173e-16 -> xyz=0.00050000000000022942759 -0.036224999999999812905 0.019550000000000553046 rpy=-1.570796326794896558 -2.2055201956572090666e-25 -2.8950564132886956449e-25
- joint right_hip_pitch: limit lower=-0.52359877559829881566 upper=1.570796326794896558 effort=1 velocity=20 -> lower=-0.52359877559829881566 upper=1.2217304763960306069 effort=1 velocity=20; origin xyz=-0.074149999999999993694 -2.0816681711721685133e-17 0.035110000000000009257 rpy=-2.1823850769468260177e-17 1.5707963267948927832 0 -> xyz=-0.074149999999999771649 5.1732706660145844069e-16 0.035110000000000037013 rpy=-6.1899281068357555747e-22 1.570796326794896336 0
- joint right_hip_roll: origin xyz=0.019050000000005999634 2.9060087669563472446e-14 -0.046014999999998154601 rpy=-1.570796326794797082 -7.3141829490872532251e-14 1.5707963267946682961 -> xyz=0.019050000000008570494 4.0564773762241657096e-14 -0.046015000000004170622 rpy=-1.5707963267947786523 -8.9077711856609251111e-14 1.5707963267946440933
- joint right_hip_yaw: origin xyz=-0.056394334796664107035 -0.041397233554676490797 0.024395090932713945492 rpy=-5.7479562369434986172e-14 0.021825623709755558738 3.5607454337323585543e-13 -> xyz=-0.018999999999998431338 -0.03500000000000151601 0.045940938812377415945 rpy=-5.7327222785292536251e-16 -2.1926904736366604217e-14 -2.7755575616618406396e-16
- joint right_knee: origin xyz=-1.360023205165816762e-15 0.07864999999999899849 0.036999999999998534062 rpy=3.141592653589793116 -5.3042305426499207572e-15 1.0017539295583627067e-13 -> xyz=1.3877787807814456755e-17 0.078649999999999137268 0.036999999999999574896 rpy=3.141592653589793116 -5.3297228769912622595e-22 -2.2267995332275346432e-26
- joint trunk_frame: origin xyz=-0.060471084556686989508 -0.0063972335546741820184 0.066744147727335195741 rpy=-6.3086333636868837384e-14 0.021825623709755163221 1.3209498708375492755e-13 -> xyz=-0.024000000000000760308 -2.4112656316077618612e-16 0.088190938812376745704 rpy=-1.4062102177136726269e-16 -9.4252837597218562265e-17 7.8061435390716270015e-33

Commit message: update

File: awd/data/assets/mini2_bdx/mini2_bdx.urdf (robot description, URDF)
Before this commit: robot onshape, 21 links, 20 joints
Joints:
- joint head_pitch: limit lower=-0.785398163397448279 upper=0.785398163397448279 effort=1 velocity=20 -> lower=-0.785398163397448279 upper=0.785398163397448279 effort=100 velocity=100
- joint head_roll: limit lower=-0.52359877559829881566 upper=0.52359877559829881566 effort=1 velocity=20 -> lower=-0.52359877559829881566 upper=0.52359877559829881566 effort=100 velocity=100
- joint head_yaw: limit lower=-2.7925268031909271649 upper=2.7925268031909271649 effort=1 velocity=20 -> lower=-2.7925268031909271649 upper=2.7925268031909271649 effort=100 velocity=100
- joint left_ankle: limit lower=-1.570796326794896558 upper=1.570796326794896558 effort=1 velocity=20 -> lower=-1.570796326794896558 upper=1.570796326794896558 effort=100 velocity=100
- joint left_antenna: limit lower=-1.570796326794896558 upper=1.570796326794896558 effort=1 velocity=20 -> lower=-1.570796326794896558 upper=1.570796326794896558 effort=100 velocity=100
- joint left_hip_pitch: limit lower=-1.2217304763960306069 upper=0.52359877559829881566 effort=1 velocity=20 -> lower=-1.2217304763960306069 upper=0.52359877559829881566 effort=100 velocity=100
- joint left_hip_roll: limit lower=-0.43633231299858238339 upper=0.43633231299858238339 effort=1 velocity=20 -> lower=-0.43633231299858238339 upper=0.43633231299858238339 effort=100 velocity=100
- joint left_hip_yaw: limit lower=-0.52359877559829881566 upper=0.52359877559829881566 effort=1 velocity=20 -> lower=-0.52359877559829881566 upper=0.52359877559829881566 effort=100 velocity=100
- joint left_knee: limit lower=-1.570796326794896558 upper=1.570796326794896558 effort=1 velocity=20 -> lower=-1.570796326794896558 upper=1.570796326794896558 effort=100 velocity=100
- joint neck_pitch: limit lower=-0.34906585039886589561 upper=1.1344640137963142301 effort=1 velocity=20 -> lower=-0.34906585039886589561 upper=1.1344640137963142301 effort=100 velocity=100
- joint right_ankle: limit lower=-1.570796326794896558 upper=1.570796326794896558 effort=1 velocity=20 -> lower=-1.570796326794896558 upper=1.570796326794896558 effort=100 velocity=100
- joint right_antenna: limit lower=-1.570796326794896558 upper=1.570796326794896558 effort=1 velocity=20 -> lower=-1.570796326794896558 upper=1.570796326794896558 effort=100 velocity=100
- joint right_hip_pitch: limit lower=-0.52359877559829881566 upper=1.2217304763960306069 effort=1 velocity=20 -> lower=-0.52359877559829881566 upper=1.2217304763960306069 effort=100 velocity=100
- joint right_hip_roll: limit lower=-0.43633231299858238339 upper=0.43633231299858238339 effort=1 velocity=20 -> lower=-0.43633231299858238339 upper=0.43633231299858238339 effort=100 velocity=100
- joint right_hip_yaw: limit lower=-0.52359877559829881566 upper=0.52359877559829881566 effort=1 velocity=20 -> lower=-0.52359877559829881566 upper=0.52359877559829881566 effort=100 velocity=100
- joint right_knee: limit lower=-1.570796326794896558 upper=1.570796326794896558 effort=1 velocity=20 -> lower=-1.570796326794896558 upper=1.570796326794896558 effort=100 velocity=100
